Commit message: navigation worked Need landing

File: src/dji_m100_description/urdf/dji_m100.urdf.xacro (robot description, xacro)
@@ -7,4 +7,6 @@
 	<xacro:include filename="$(find dji_m100_description)/urdf/guidance.urdf.xacro" />
     <xacro:dji_m100_guidance_macro/>
+    <xacro:include filename="$(find dji_m100_description)/urdf/lidar.urdf.xacro" />
+    <xacro:lidar_macro/>
     <!--<xacro:include filename="$(find dji_m100_description)/urdf/gimbal.urdf.xacro" />-->
     <!--<xacro:dji_m100_gimbal />-->

File: src/dji_m100_description/urdf/guidance.urdf.xacro (robot description, xacro)
@@ -116,4 +116,100 @@
       		</sensor>
     	</gazebo>
+    	<!-- ********************************************* -->
+    	<!-- Guidance Down Link -->
+	    <joint name="guidance_down_joint" type="fixed">
+	      	<origin xyz="0 0.035 -0.3" rpy="0 ${pi/2} 0 "/>
+	      	<parent link="guidance_base"/>
+	      	<child link="guidance_down_base"/>
+	    </joint>
+	    <link name="guidance_down_base">
+		    <collision>
+		    	<origin xyz="0 0 0" rpy="0 0 0"/>
+		        <geometry>
+		        	<box size="${box_size} ${box_size*2} ${box_size}"/>
+		        </geometry>
+		      </collision>
+		      <visual>
+		        <origin xyz="0 0 0" rpy="0 0 0"/>
+		        <geometry>
+		          	<box size="${box_size} ${box_size*2} ${box_size}"/>
+		        </geometry>
+		        <material name="red"/>
+		      </visual>
+		    <inertial>
+		        <mass value="1e-5" />
+		        <origin xyz="0 0 0" rpy="0 0 0"/>
+		        <inertia ixx="1e-6" ixy="0" ixz="0" iyy="1e-6" iyz="0" izz="1e-6" />
+		    </inertial>
+	    </link>
+	    <!-- Guidance Down Optical Link -->
+	    <!-- Rotate frame from x-forward to z-froward camera coords-->
+	    <joint name="guidance_down_optical_joint" type="fixed">
+	      	<origin xyz="0 0 0" rpy="${-pi/2} 0 ${-pi/2}"/>
+	      	<parent link="guidance_down_base"/>
+	      	<child link="guidance_down"/>
+	    </joint>
+	    <link name="guidance_down">
+  		</link>
+  		<gazebo reference="guidance_down_base">
+	      	<!-- Sensor Parameter -->
+	      	<sensor type="multicamera" name="stereo_camera">
+		        <update_rate>30</update_rate>
+		        <camera name="left">
+		          <horizontal_fov>1.209513</horizontal_fov>
+		          <image>
+		            <width>320</width>
+		            <height>240</height>
+		            <format>R8G8B8</format>
+		          </image>
+		          <clip>
+		            <near>0.02</near>
+		            <far>300</far>
+		          </clip>
+		          <noise>
+		            <type>gaussian</type>
+		            <mean>0.0</mean>
+		            <stddev>0.007</stddev>
+		          </noise>
+		        </camera>
+		        <camera name="right">
+		          <pose>0 -0.07 0 0 0 0</pose>
+		          <horizontal_fov>1.209513</horizontal_fov> <!--image_width/(2*tan(hfov_radian/2))-->
+		          <image>
+		            <width>320</width>
+		            <height>240</height>
+		            <format>R8G8B8</format>
+		          </image>
+		          <clip>
+		            <near>0.02</near>
+		            <far>300</far>
+		          </clip>
+		          <noise>
+		            <type>gaussian</type>
+		            <mean>0.0</mean>
+		            <stddev>0.007</stddev>
+		          </noise>
+		        </camera>
+	        	<!--Plugin Parameter-->
+	        	<plugin name="stereo_camera_controller" filename="libgazebo_ros_multicamera.so">
+		          <alwaysOn>true</alwaysOn>
+		          <updateRate>0.0</updateRate>
+		          <cameraName>guidance_down</cameraName>
+		          <imageTopicName>image_raw</imageTopicName>
+		          <cameraInfoTopicName>camera_info</cameraInfoTopicName>
+		          <frameName>guidance_down</frameName>
+		          <Cx>157.0</Cx>
+		          <Cy>122.5</Cy>
+		          <focalLength>231.501514</focalLength>
+		          <hackBaseline>0.1532</hackBaseline>
+		          <distortionK1>-0.019359</distortionK1>
+		          <distortionK2>-0.002195</distortionK2>
+		          <distortionT1>-0.001779</distortionT1>
+		          <distortionT2>0.000335</distortionT2>
+		          <distortionK3>0.0</distortionK3>
+	        	</plugin>
+      		</sensor>
+    	</gazebo>
+    	<!-- ********************************************* -->
   	</xacro:macro>
 </robot>
