Commit message: Integrated landing

File: src/dji_m100_description/urdf/guidance.urdf.xacro (robot description, xacro)
@@ -26,7 +26,7 @@
 	      	<origin xyz="0.1 0.035 0" rpy="0 0 0"/>
 	      	<parent link="guidance_base"/>
-	      	<child link="guidance_front"/>
-	    </joint>
-	    <link name="guidance_front">
+	      	<child link="guidance_front_base"/>
+	    </joint>
+	    <link name="guidance_front_base">
 		    <collision>
 		    	<origin xyz="0 0 0" rpy="0 0 0"/>
@@ -52,10 +52,10 @@
 	    <joint name="camera_optical_joint" type="fixed">
 	      	<origin xyz="0 0 0" rpy="${-pi/2} 0 ${-pi/2}"/>
-	      	<parent link="guidance_front"/>
-	      	<child link="guidance_front_optical"/>
-	    </joint>
-	    <link name="guidance_front_optical">
+	      	<parent link="guidance_front_base"/>
+	      	<child link="guidance_front"/>
+	    </joint>
+	    <link name="guidance_front">
   		</link>
-  		<gazebo reference="guidance_front">
+  		<gazebo reference="guidance_front_base">
 	      	<!-- Sensor Parameter -->
 	      	<sensor type="multicamera" name="stereo_camera">
@@ -103,5 +103,5 @@
 		          <imageTopicName>image_raw</imageTopicName>
 		          <cameraInfoTopicName>camera_info</cameraInfoTopicName>
-		          <frameName>guidance_front_optical</frameName>
+		          <frameName>guidance_front</frameName>
 		          <Cx>157.0</Cx>
 		          <Cy>122.5</Cy>
@@ -119,5 +119,6 @@
     	<!-- Guidance Down Link -->
 	    <joint name="guidance_down_joint" type="fixed">
-	      	<origin xyz="0 0.035 -0.3" rpy="0 ${pi/2} 0 "/>
+	      	<!-- <origin xyz="0 0.035 -0.3" rpy="0 ${pi/2} 0 "/> -->
+	      	<origin xyz="0 0 -0.3" rpy="0 ${pi/2} 0 "/>
 	      	<parent link="guidance_base"/>
 	      	<child link="guidance_down_base"/>
@@ -174,5 +175,5 @@
 		        </camera>
 		        <camera name="right">
-		          <pose>0 -0.07 0 0 0 0</pose>
+		          <pose>0 0.07 0 0 0 0</pose>
 		          <horizontal_fov>1.209513</horizontal_fov> <!--image_width/(2*tan(hfov_radian/2))-->
 		          <image>
